File: Aurora/Aurora.kicad_sch (KiCad schematic)
At the start: 37 parts, among them J1 UJ20-C-H-C-3-SMT-TR, U1 STM32H757BITx, U2 USBLC6-2SC6, U3 TLV76733DRVx

Commit message: added 7.4->5v regulator for battery
Parts:
- added BT1: 7.4V, symbol Device:Battery
- added C30: 10uF, symbol Device:C_Small
- added C31: 100nF, symbol Device:C_Small
- added C32, C33: 22uF, symbol Device:C_Small
- added L1: 4.7uH, symbol Device:L
- added U4: AP63205WU-7, SOIC_05WU-7_DIO, symbol 2025-09-13_17-48-58:AP63205WU-7
Connections:
- net USB_3V3 is gone; now on net 3V3: C1.2, C10.2, C11.2, C12.2, C13.2, C14.2, C15.2, C16.2, C17.2, C18.2, C2.2, C21.2, C26.2, C29.1, C3.2, C4.2, C5.2, C6.2, C7.2, C8.2, C9.2, R3.1, U1.100 (VDD), U1.108 (VDD), U1.114 (VDD), U1.117 (VDD), U1.133 (VDD), U1.141 (VDD33_USB), U1.155 (VDD), U1.161 (VDD), U1.17 (VDD), U1.179 (VDD), U1.187 (VDD), U1.208 (VDD), U1.29 (VDD), U1.49 (VDD), U1.56 (VDD), U1.7 (VDD), U1.74 (VDD), U1.8 (VBAT), U1.80 (VDD), U3.1 (OUT)
- net GND: now also BT1.2 (-), C30.1, C32.1, L1.1, U4.1 (FB), U4.4 (GND)
- net +3.3V renamed 3V3
- new net: BT1.1 (+), C30.2, U4.2 (EN), U4.3 (VIN)
- new net: C31.1, L1.2, U4.5 (SW)
- new net: C31.2, U4.6 (BST)
- new net: C32.2, C33.1
- new net BATT_5V: C33.2
Other:
- note added: "--Voltage Regulator-- All values and wiring from datasheet See typical application circuit on pg. 2"
- note added: "5V-Battery"
- note added: "USB"
- moved on the sheet: C27, C28, C29, J1, R1, R2, R3, R4, U2, U3

Commit message: power multiplexer
Parts:
- removed C30: 10uF, symbol Device:C_Small
- removed C31: 100nF, symbol Device:C_Small
- removed C32, C33: 22uF, symbol Device:C_Small
- removed L1: 4.7uH, symbol Device:L
- removed U3: TLV76733DRVx, Package_SON:WSON-6-1EP_2x2mm_P0.65mm_EP1x1.6mm_ThermalVias, symbol Regulator_Linear:TLV76733DRVx
- removed U4: AP63205WU-7, SOIC_05WU-7_DIO, symbol 2025-09-13_17-48-58:AP63205WU-7
- added R5, R7: 5kR, symbol Device:R_Small
- added R6: 23k7, symbol Device:R_Small
- added U3: TPS2121RUXR, footprints1:RUX0012A, symbol 2025-09-13_19-11-07:TPS2121RUXR
- C28: value 1uF -> 100nF
- C29: value 4.7uF -> 0.01uF
- R3: value 500kR -> 22k1
- R4: value 160kR -> 41k2
Connections:
- net 3V3: no longer C29.1, R3.1
- net GND: now also R3.2, R5.2, R7.2, U3.12 (GND), U3.3 (CP2), U3.6 (PR1), U3.9 (ST); no longer C28.2, R4.2
- net USB_VBUS: now also R6.1, U3.7 (IN1); no longer C28.1
- net at BT1.1 (+): now also R4.1, U3.2 (IN2)
- new net: R3.1, U3.10 (ILM)
- new net: C29.1, U3.11 (SS)
- new net: R4.2, R5.1, U3.4 (OV2)
- new net: R6.2, R7.1, U3.5 (OV1)
- new net V_OUT: C28.1, U3.1 (OUT)
- no-connect marks 2 -> 3
Other:
- note added: "5V-USB"
- note added: "Power MUX"
- note removed: "--Voltage Regulator-- All values and wiring from datasheet See typical application circuit on pg. 2"
- note removed: "--Voltage Regulator-- Input&Enable pins connected to 5V Input/output capacitor values determined from datasheet 4.7uF Capacitor chosen for manufacturing convenience Resistor values set up to give output voltage of 3.3V Specific values from datasheet"
- note removed: "5V-Battery"
- note removed: "USB"
- moved on the sheet: C27, J1, R1, R2, U2

Commit message: 3.3v regulator
Parts:
- removed BT1: 7.4V, symbol Device:Battery
- added C30: 10uF, symbol Device:C_Small
- added C31, C32: 22uF, symbol Device:C_Small
- added C33: 100uF, symbol Device:C_Small
- added L1: 3.3uH, symbol Device:L
- added U4: AP63203QWU-7, TSOT26_DIO, symbol 2025-09-13_20-10-09:AP63203QWU-7
Connections:
- net 3V3: now also C32.2, L1.2, U4.1 (FB)
- net GND: now also C23.1, C24.1, C25.1, C30.1, C31.1, U4.4 (GND)
- net V_OUT: now also C30.2, U4.2 (EN), U4.3 (VIN)
- net 7.4V: now reaches R4.1, U3.2 (IN2)
- new net: C31.2, C32.1
- new net: C33.2, L1.1, U4.5 (SW)
- new net: C33.1, U4.6 (BST)
Other:
- note added: "--3.3V Regulator-- Takes in output from Power MUX and regulates it down to 3.3V All wiring and resistor/capacitor values taken from datasheet"
- note added: "--Power MUX-- USB power = Input 1, Batt = Input 2 Wired such that when USB is plugged in, switches from Battery to USB Resistor/Capacitor values and wiring taken from datasheet"
- note added: "->"
- note added: "3V3 Regulator"
- note added: "This 41.2 ohm resistor was calculated using intended current and provided voltage (OHMS LAW （⊙ｏ⊙）)"
