File: Aurora/Aurora.kicad_sch (KiCad schematic)
At the start: 54 parts, among them J1 UJ20-C-H-C-3-SMT-TR, U1 STM32H757BITx, U2 USBLC6-2SC6, U3 TPS2121RUXR, U4 AP63203QWU-7, U5 ICM-45686, U6 ICM-42688-P

Commit message: did some work on gyroscope, wired up IMU
Parts:
- added C38, C39, C40: 100nF, symbol Device:C_Small
- added C41, C42: 22pF, symbol Device:C_Small
- added R10, R9: 2.2kR, symbol Device:R_Small
- added R8: 10kR, symbol Device:R_Small
- added U7: BNO085, BNO085:IC_BNO085, symbol BNO085:BNO085
- added Y1: ASEK-32.768KHZ-L-R-T, ASEK-32.768KHZ-L-R-T:XTAL_ASEK-32.768KHZ-L-R-T, symbol ASEK-32.768KHZ-L-R-T:ASEK-32.768KHZ-L-R-T
Connections:
- net 3V3: now also C38.2, C39.2, R10.2, R8.2, R9.2, U7.28 (VDDIO), U7.3 (VDD), U7.5 (PS1)
- net GND: now also C38.1, C39.1, C40.2, C41.2, C42.1, U7.2 (GND), U7.25 (GNDIO), Y1.2 (GND/CASE)
- net FSYNC/CLKIN: now reaches U5.9 (INT2/FSYNC/CLKIN)
- new net: R9.1, U7.16 (ENV_SDA)
- new net: C40.1, U7.9 (CAP)
- new net: R10.1, U7.15 (ENV_SCL)
- new net: U7.1 (RESV_NC), U7.12 (RESV_NC), U7.13 (RESV_NC), U7.21 (RESV_NC), U7.22 (RESV_NC), U7.23 (RESV_NC), U7.24 (RESV_NC), U7.7 (RESV_NC), U7.8 (RESV_NC)
- new net BNO_BOOTN: R8.1, U7.4 (~{BOOT})
- new net BNO_CLKSEL0: U7.10 (CLKSEL0)
- new net BNO_NRST: U7.11 (~{RST})
- new net BNO_WAKE/PS0: U7.6 (PS0/WAKE)
- new net STM_CLK: U7.19 (H_SCL/SCK/RX)
- new net STM_CSN: U7.18 (~{H_CS})
- new net STM_INTN: U7.14 (~{H_INT})
- new net STM_MISO: U7.20 (H_SDA/H_MISO/TX)
- new net STM_MOSI: U7.17 (SA0/H_MOSI)
- new net XIN_32: C41.1, U7.27 (XIN32), Y1.4 (VDD)
- new net XOUT_32: C42.2, U7.26 (XOUT32/CLKSEL1), Y1.3 (OUTPUT)
- no-connect marks 7 -> 9
Other:
- note added: "--32.768kHz Oscillator-- Oscillator for BNO085 Pin 1 left floating because we are not using it; see datasheet"
- note added: "32.768kHz"

Commit message: wired up ICM-45686, ICM-42688, and Barometer to STM
Parts:
- added C43, C46: 100nF, symbol Device:C_Small
- added C44: 10nF, symbol Device:C_Small
- added C45: 2.2uF, symbol Device:C_Small
- added R11, R12, R13: 10kR, symbol Device:R_Small
Connections:
- net AP_CLK is gone; now on net ICM456_CLK: U5.13 (AP_SCL/AP_SCLK)
- net AP_SDIO is gone; now on net ICM456_MOSI: U5.14 (AP_SDA/AP_SDIO/AP_SDI)
- net AP_SDO is gone; now on net ICM456_MISO: U5.1 (AP_SDO/AP_AD0)
- net STM_CLK is gone; now on net BNO_CLK: U7.19 (H_SCL/SCK/RX)
- net STM_MISO is gone; now on net BNO_MISO: U7.20 (H_SDA/H_MISO/TX)
- net STM_MOSI is gone; now on net BNO_MOSI: U7.17 (SA0/H_MOSI)
- net 3V3: now also Barometer-(U7).1 (VDDIO), Barometer-(U7).10 (VDD), Micro-SD-Socket-(J2).P4 (VDD1), U6.5 (VDDIO), U6.8 (VDD), C43.2, C44.1, C45.2, C46.2, R11.1, R12.1, R13.2
- net GND: now also Barometer-(U7).3 (VSS/GND), Barometer-(U7).8 (VSS/GND), Barometer-(U7).9 (VSS/GND), C28.2, Micro-SD-Socket-(J2).P10 (COVER_GND), Micro-SD-Socket-(J2).P11 (COVER_GND__1), Micro-SD-Socket-(J2).P12 (COVER_GND__2), Micro-SD-Socket-(J2).P13 (COVER_GND__3), Micro-SD-Socket-(J2).P14 (COVER_GND__4), Micro-SD-Socket-(J2).P17 (VSS__1), Micro-SD-Socket-(J2).P20 (VSS__2), Micro-SD-Socket-(J2).P23 (VSS__3), Micro-SD-Socket-(J2).P6 (VSS), U6.11 (RESV_11), U6.6 (GND), C43.1, C44.2, C45.1, C46.1
- net ICM456_INT: now reaches U5.4 (INT1/INT)
- net BMP_CLK: now reaches U1.1 (PE2)
- net BMP_CLK: now also Barometer-(U7).2 (SCK/SCL)
- net ICM426_CLK: now reaches U1.167 (PC10)
- net ICM426_CLK: now also U6.13 (AP_SCL/AP_SCLK)
- net ICM426_MISO: now reaches U1.168 (PC11)
- net ICM426_MISO: now also U6.1 (AP_SDO/AP_AD0)
- net BNO_MOSI: now reaches U1.39 (PC1)
- net BMP_MISO: now reaches U1.4 (PE5)
- net BMP_MISO: now also Barometer-(U7).5 (SDO/DNC/SA0)
- net BNO_MISO: now reaches U1.40 (PC2_C)
- net BMP_MOSI: now reaches U1.5 (PE6)
- net BMP_MOSI: now also Barometer-(U7).4 (SDI/SDO/SDA)
- net ICM456_CLK: now reaches U1.58 (PA5)
- net ICM456_MISO: now reaches U1.59 (PA6)
- net ICM456_MOSI: now reaches U1.60 (PA7)
- net ICM426_MOSI: now reaches U1.65 (PB2)
- net ICM426_MOSI: now also U6.14 (AP_SDA/AP_SDIO/AP_SDI)
- net BNO_CLK: now reaches U1.87 (PB10)
- net ICM426_CS: now reaches U6.12 (AP_CS)
- net ICM426_CS: now also R12.2
- net ICM426_INT: now reaches U6.4 (INT1/INT)
- net 1V8: now reaches Micro-SD-Socket-(J2).P15 (VDD2)
- net BMP_CS: now reaches Barometer-(U7).6 (~{CS})
- net BMP_CS: now also R13.1
- net BMP_INT: now reaches Barometer-(U7).7 (INT/DNC)
- net AP_CS renamed ICM456_CS
- net ICM456_CS: now also R11.2
- net FSYNC/CLKIN: no longer names the net of U5.9 (INT2/FSYNC/CLKIN)
- no-connect marks 9 -> 15
Other:
- note added: "--Barometer-- Resistors/capacitors from datasheet (Fig 24)/Other designs"
- note added: "--ICM-42688-- Gyroscope Resistors/capacitors from datasheet (Fig 7)/Other designs"
- note added: "--ICM-45686-- Another IMU Resistors/capacitors from datasheet/other designs"
- note added: "--IMU-- Reference Fig. 1-20 in datasheet, that's where all this comes from"
- note added: "Barometer"
- note added: "ICM-42688-P"
- note added: "ICM-45686"
- note added: "IMU"
- moved on the sheet: Barometer-(U7), C1, C10, C11, C12, C13, C14, C15, C16, C17, C18, C19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

Commit message: SD Card wired up
Parts:
- removed C22, C24, C25, C34, C35: 100nF, symbol Device:C_Small
- removed C23: 4.7uF, symbol Device:C_Small
- removed Micro-SD-Socket-(J2): MSD4-3-A, MSD4_3_A:CUI_MSD4-3-A, symbol MSD4-3-A:MSD4-3-A
- added J2: DM3AT-SF-PEJM5, DM3AT-SF-PEJM5:HRS_DM3AT-SF-PEJM5, symbol DM3AT-SF-PEJM5:DM3AT-SF-PEJM5
- added R14: 10kR, symbol Device:R_Small
- added SW1: PCM12SMTR, PCM12SMTR:SW_PCM12SMTR, symbol PCM12SMTR:PCM12SMTR
Connections:
- net 3V3: now also C19.2, C20.2, U1.43 (VREF+), U1.44 (VDDA), J2.4 (VDD), SW1.1; no longer U1.20 (VDDSMPS)
- net GND: now also J2.6 (VSS), J2.P1 (SHIELD), J2.P2 (SHIELD__1), J2.P3 (SHIELD__2), J2.P4 (SHIELD__3), SW1.3, SW1.S1 (SHIELD), SW1.S2 (SHIELD__1), SW1.S3 (SHIELD__2), SW1.S4 (SHIELD__3)
- net ICM426_CLK: now also U1.189 (PB3); no longer U1.167 (PC10)
- net ICM426_MISO: now also U1.190 (PB4); no longer U1.168 (PC11)
- net SD_DAT0: now reaches U1.144 (PC8)
- net SD_DAT0: now also J2.7 (DAT0)
- net SD_DAT1: now reaches U1.145 (PC9)
- net SD_DAT1: now also J2.8 (DAT1)
- net SD_CLK: now reaches U1.169 (PC12)
- net SD_CLK: now also J2.5 (CLK)
- net SD_CMD: now reaches U1.172 (PD2)
- net SD_CMD: now also J2.3 (CMD)
- net at U1.194 (BOOT0): now also R14.1
- net +5V: no longer names the net of U1.140 (VDD50_USB)
- new net: R14.2, SW1.2
- new net SD_DAT2: J2.1 (DAT2), U1.167 (PC10)
- new net SD_DAT3: J2.2 (CD/DAT3), U1.168 (PC11)
- no-connect marks 15 -> 17
Other:
- note added: "--Barometer-- Resistors/capacitors from datasheet (Fig 24)/Other designs SPI 4"
- note added: "--ICM-42688-- Gyroscope Resistors/capacitors from datasheet (Fig 7)/Other designs SPI 3"
- note added: "--ICM-45686-- Another IMU Resistors/capacitors from datasheet/other designs SPI 1"
- note added: "--IMU-- Reference Fig. 1-20 in datasheet, that's where all this comes from SPI2"
- note added: "SD Card"
- note removed: "--Barometer-- Resistors/capacitors from datasheet (Fig 24)/Other designs"
- note removed: "--ICM-42688-- Gyroscope Resistors/capacitors from datasheet (Fig 7)/Other designs"
- note removed: "--ICM-45686-- Another IMU Resistors/capacitors from datasheet/other designs"
- note removed: "--IMU-- Reference Fig. 1-20 in datasheet, that's where all this comes from"
- moved on the sheet: C1, C10, C11, C12, C13, C14, C15, C16, C17, C18, C19, C2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

Commit message: Hooked up XB radio, began breaking out the rest of the SPI and UART pins
Parts:
- removed R13: 10kR, symbol Device:R_Small
- added U8: XBP9X-DMUS-021, XBP9X-DMUS-021:DIP2200W51P200L3294H279Q20P, symbol XBP9X-DMUS-021:XBP9X-DMUS-021
Connections:
- net 3V3: now also U8.1 (VCC)
- net GND: now also U8.10 (GND)
- net XB_TX: now reaches U1.13 (PI9)
- net XB_TX: now also U8.2 (DOUT/DIO13)
- net SPI6_MISO: now reaches U1.183 (PG12)
- net SPI6_CLK: now reaches U1.184 (PG13)
- net SPI6_MOSI: now reaches U1.185 (PG14)
- net SPI5_CLK: now reaches U1.31 (PF7)
- net SPI5_MISO: now reaches U1.32 (PF8)
- net SPI5_MOSI: now reaches U1.33 (PF9)
- net XB_RX: now reaches U1.45 (PA0)
- net XB_RX: now also U8.3 (DIN/NCONFIG/DIO14)
- net BMP_CLK renamed B/R_CLK
- net B/R_CLK: now also U8.18 (AD2/DIO2/SPI_CLK)
- net BMP_MISO renamed B/R_MISO
- net B/R_MISO: now also U8.4 (DIO12/SPI_MISO)
- net BMP_MOSI renamed B/R_MOSI
- net B/R_MOSI: now also U8.11 (DIO4/SPI_MOSI)
- new net XBP_ATTN: U8.19 (AD1/DIO1/SPI_NATTN)
- new net XBP_CS: U8.17 (AD3/DIO3/SPI_NSSEL)
- no-connect marks 17 -> 26
Other:
- note added: "*"
- note added: "* NOTE: On the MCU, the XB_TX line RECEIVES data from the XB, while the XB_RX line SENDS data to the XB. Follow the direction the flag points"
- note added: "--XB Radio-- Using SPI and UART protocols SPI 4/UART 4"
- note added: "XB Radio"

Commit message: lots of changes; sensors, LEDs, screw terminal blocks
Parts:
- removed Barometer-(U7): BMP390L, BMP390L:XDCR_BMP390L, symbol BMP390L:BMP390L
- removed C1, C10, C11, C12, C13, C14, C15, C16, C17, C18, C19, C2, C26, C27, C28, C3, C36, C37, C38, C39, C4, C40, C43, C46, C5, C6, C7, C8, C9: 100nF, symbol Device:C_Small
- removed C20: 1uF, symbol Device:C_Small
- removed C21: 4.7uF, symbol Device:C_Small
- removed C29: 0.01uF, symbol Device:C_Small
- removed C30: 10uF, symbol Device:C_Small
- removed C31, C32: 22uF, symbol Device:C_Small
- removed C33: 100uF, symbol Device:C_Small
- removed C41, C42: 22pF, symbol Device:C_Small
- removed C44: 10nF, symbol Device:C_Small
- removed C45: 2.2uF, symbol Device:C_Small
- removed J1: UJ20-C-H-C-3-SMT-TR, UJ20-C-H-C-3-SMT-TR (1):CUI_UJ20-C-H-C-3-SMT-TR, symbol UJ20-C-H-C-3-SMT-TR:UJ20-C-H-C-3-SMT-TR
- removed J2: DM3AT-SF-PEJM5, DM3AT-SF-PEJM5:HRS_DM3AT-SF-PEJM5, symbol DM3AT-SF-PEJM5:DM3AT-SF-PEJM5
- removed L1: 3.3uH, symbol Device:L
- removed R1, R2: 5k1, symbol Device:R_Small
- removed R10, R9: 2.2kR, symbol Device:R_Small
- removed R11, R12, R14, R8: 10kR, symbol Device:R_Small
- removed R3: 22k1, symbol Device:R_Small
- removed R4: 41k2, symbol Device:R_Small
- removed R5, R7: 5kR, symbol Device:R_Small
- removed R6: 23k7, symbol Device:R_Small
- removed SW1: PCM12SMTR, PCM12SMTR:SW_PCM12SMTR, symbol PCM12SMTR:PCM12SMTR
- removed U1: STM32H757BITx, Package_QFP:LQFP-208_28x28mm_P0.5mm, symbol MCU_ST_STM32H7:STM32H757BITx
- removed U2: USBLC6-2SC6, USBLC6_2SC6:SOT95P280X145-6N, symbol USBLC6-2SC6:USBLC6-2SC6
- removed U3: TPS2121RUXR, footprints1:RUX0012A, symbol 2025-09-13_19-11-07:TPS2121RUXR
- removed U4: AP63203QWU-7, TSOT26_DIO, symbol 2025-09-13_20-10-09:AP63203QWU-7
- removed U5: ICM-45686, ICM_45686:IC_ICM-45686, symbol ICM-45686:ICM-45686
- removed U6: ICM-42688-P, ICM_42688_P:PQFN50P300X250X97-14N, symbol ICM-42688-P:ICM-42688-P
- removed U7: BNO085, BNO085:IC_BNO085, symbol BNO085:BNO085
- removed U8: XBP9X-DMUS-021, XBP9X-DMUS-021:DIP2200W51P200L3294H279Q20P, symbol XBP9X-DMUS-021:XBP9X-DMUS-021
- removed Y1: ASEK-32.768KHZ-L-R-T, ASEK-32.768KHZ-L-R-T:XTAL_ASEK-32.768KHZ-L-R-T, symbol ASEK-32.768KHZ-L-R-T:ASEK-32.768KHZ-L-R-T
Connections:
- no-connect marks 26 -> 0
Other:
- added sheet Chips (Chips.kicad_sch)
- added sheet Terminal Blocks (pyros.kicad_sch)
- added sheet Top (top.kicad_sch)
- note removed: "*"
- note removed: "* NOTE: On the MCU, the XB_TX line RECEIVES data from the XB, while the XB_RX line SENDS data to the XB. Follow the direction the flag points"
- note removed: "--3.3V Regulator-- Takes in output from Power MUX and regulates it down to 3.3V All wiring and resistor/capacitor values taken from datasheet"
- note removed: "--32.768kHz Oscillator-- Oscillator for BNO085 Pin 1 left floating because we are not using it; see datasheet"
- note removed: "--Barometer-- Resistors/capacitors from datasheet (Fig 24)/Other designs SPI 4"
- note removed: "--ESD-- Capacitor value determined from other designs Don't ask me what it does"
- note removed: "--ICM-42688-- Gyroscope Resistors/capacitors from datasheet (Fig 7)/Other designs SPI 3"
- note removed: "--ICM-45686-- Another IMU Resistors/capacitors from datasheet/other designs SPI 1"
- note removed: "--IMU-- Reference Fig. 1-20 in datasheet, that's where all this comes from SPI2"
- note removed: "--Power Delivery-- 3.3V rail comes from battery/USB 100nF capacitors = decoupling capacitors (1 per input pin) 4.7uF & 1uF capacitors = bulk capacitors (1 per power rail) LDOs tied to SMPS level to provide 1.2V WIP: Do we provide power to VDD50_USB?"
- note removed: "--Power MUX-- USB power = Input 1, Batt = Input 2 Wired such that when USB is plugged in, switches from Battery to USB Resistor/Capacitor values and wiring taken from datasheet"
- note removed: "--USB Connector-- +/- Diff pairs connected bc of usb-c symmetry VBUS pulled from device connected to voltage reg (5->3.3) CCs set up as a sink device to pull power from connection All lines hooked up to ESD protection"
- note removed: "--XB Radio-- Using SPI and UART protocols SPI 4/UART 4"
- note removed: "->"
- note removed: "32.768kHz"
- note removed: "3V3 Regulator"
- note removed: "5V-USB"
- note removed: "Barometer"
- note removed: "ICM-42688-P"
- note removed: "ICM-45686"
- note removed: "IMU"
- note removed: "Power MUX"
- note removed: "SD Card"
- note removed: "STM32H7"
- note removed: "This 41.2 ohm resistor was calculated using intended current and provided voltage (OHMS LAW （⊙ｏ⊙）)"
- note removed: "XB Radio"

Commit message: Add files via upload
Other:
- sheet Terminal Blocks renamed Bottom Board Terminal Blocks
Changed lines of the file:
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@@
 			(color 0 0 0 0.0000)
 		)
-		(property "Sheetname" "Terminal Blocks"
+		(property "Sheetname" "Bottom Board Terminal Blocks"
 			(at 17.78 18.3384 0)
 			(effects
