File: Aurora/Aurora.kicad_pcb (KiCad board)
At the start: 2 copper layers, 86 parts, among them J1 UJ20-C-H-C-3-SMT-TR, J10 Screw_Terminal_01x02, J11 Screw_Terminal_01x02, J12 Screw_Terminal_01x04, J13 Screw_Terminal_01x02, J14 Screw_Terminal_01x02, J15 Screw_Terminal_01x02, J2 Screw_Terminal_01x04, J4 Screw_Terminal_01x08, J5 Screw_Terminal_01x08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

Commit message: reorganization
Parts:
- added C48: 100nF, Capacitor_SMD:C_1206_3216Metric, F.Cu at (256.4, 72.5)
- added C49: 10uF, Capacitor_SMD:C_1206_3216Metric, F.Cu at (256.4, 75.9)
- added C50: 220uF, Capacitor_SMD:C_1206_3216Metric, F.Cu at (256.4, 79.2)
- added C51: 0.33uF, Capacitor_SMD:C_1206_3216Metric, F.Cu at (273.5, 110.2)
- added C52: 100nF, Capacitor_SMD:C_1206_3216Metric, F.Cu at (273.5, 113.5)
- added D2: LED, LED_SMD:LED_Cree-PLCC4_5x5mm_CW, F.Cu at (236.5, 74.2)
- added D3: LED, LED_SMD:LED_Cree-PLCC4_5x5mm_CW, F.Cu at (236.5, 81.0)
- added D4: LED, LED_SMD:LED_Cree-PLCC4_5x5mm_CW, F.Cu at (236.5, 87.8)
- added D5: WS2812B-2020, LED_SMD:LED_WS2812B-2020_PLCC4_2.0x2.0mm, F.Cu at (261.4, 72.7)
- added J16: PPPC042LFBN-RC, PPPC042LFBN_RC:SULLINS_PPPC042LFBN-RC, F.Cu at (246.9, 80.8)
- added J17: Screw_Terminal_01x04, footprints6:CONN_1715747_PXC, F.Cu at (237.8, 99.2)
- added J18: Screw_Terminal_01x04, footprints6:CONN_1715747_PXC, F.Cu at (237.8, 110.6)
- added J19: TSW-104-27-G-D, TSW_104_27_G_D:SAMTEC_TSW-104-27-G-D, F.Cu at (261.0, 103.8)
- added J20: TSW-104-27-G-D, TSW_104_27_G_D:SAMTEC_TSW-104-27-G-D, F.Cu at (261.0, 110.4)
- added J3: PPPC042LFBN-RC, PPPC042LFBN_RC:SULLINS_PPPC042LFBN-RC, F.Cu at (246.9, 74.2)
- added J4: Screw_Terminal_01x08, footprints7:CONN_1715789_PXC, F.Cu at (237.8, 54.0)
- added J5: Screw_Terminal_01x08, footprints7:CONN_1715789_PXC, F.Cu at (237.8, 65.5)
- added R13: 82R, Resistor_SMD:R_1206_3216Metric, F.Cu at (256.4, 82.6)
- added R15: 50R, Resistor_SMD:R_1206_3216Metric, F.Cu at (256.4, 85.9)
- added R16: 270R, Resistor_SMD:R_1206_3216Metric, F.Cu at (256.4, 89.2)
- added U10: ADS1115IDGS, Package_SO:TSSOP-10_3x3mm_P0.5mm, F.Cu at (274.2, 101.5)
- added U11: ADS1115IDGS, Package_SO:TSSOP-10_3x3mm_P0.5mm, F.Cu at (274.2, 106.2)
- added U12: L7805, L7805:TO255P1020X450X2000-3, F.Cu at (265.0, 96.2)
- moved U1 7.02 mm to (69.0, 60.0)
Connections:
- net 7.4V renamed Net-(D4-K)
- net MCP_SCL renamed EXP_SCL
- net MCP_SDA renamed EXP_SDA
- C27 pad 1: USB_VBUS -> Net-(C27-Pad1)
- J1 pad A4_B9: USB_VBUS -> Net-(C27-Pad1)
- J1 pad A9_B4: USB_VBUS -> Net-(C27-Pad1)
- J12 pad 1: unconnected-(J12-Pin_1-Pad1) -> GND
- J12 pad 2: unconnected-(J12-Pin_2-Pad2) -> GND
- J12 pad 3: unconnected-(J12-Pin_3-Pad3) -> GND
- J12 pad 4: unconnected-(J12-Pin_4-Pad4) -> GND
- J13 pad 1: I2C2_SCL -> I2C4_SCL
- J13 pad 2: I2C2_SDA -> I2C4_SDA
- J14 pad 1: I2C3_SCL -> I2C4_SCL
- J14 pad 2: I2C3_SDA -> I2C4_SDA
- J9 pad 1: unconnected-(J9-Pin_1-Pad1) -> 3.3V
- J9 pad 2: unconnected-(J9-Pin_2-Pad2) -> 5V
- J9 pad 3: unconnected-(J9-Pin_3-Pad3) -> 5V
- J9 pad 4: unconnected-(J9-Pin_4-Pad4) -> 5V
- U1 pad 105: unconnected-(U1-PD8-Pad105) -> HDR_GPIO1
- U1 pad 106: unconnected-(U1-PD9-Pad106) -> HDR_GPIO2
- U1 pad 107: unconnected-(U1-PD10-Pad107) -> HDR_GPIO3
- U1 pad 110: unconnected-(U1-PD11-Pad110) -> HDR_GPIO4
- U1 pad 111: unconnected-(U1-PD12-Pad111) -> HDR_GPIO5
- U1 pad 112: unconnected-(U1-PD13-Pad112) -> HDR_GPIO6
- U1 pad 115: unconnected-(U1-PD14-Pad115) -> HDR_GPIO7
- U1 pad 116: unconnected-(U1-PD15-Pad116) -> HDR_GPIO8
- U1 pad 22: I2C2_SDA -> ADC1_SDA
- U1 pad 23: I2C2_SCL -> ADC1_SCL
- U1 pad 72: unconnected-(U1-PG0-Pad72) -> Net-(D5-DIN)
- U1 pad 93: I2C3_SCL -> ADC2_SCL
- U1 pad 94: I2C3_SDA -> ADC2_SDA
- U2 pad 5: USB_VBUS -> Net-(C27-Pad1)
- U8 pad 6: unconnected-(U8-DIO10/PWM0-Pad6) -> Net-(U8-DIO10/PWM0)
- U9 pad 9: 3V3 -> 5V
