File: Aurora_new/Aurora.kicad_pcb (KiCad board)
At the start: 2 copper layers, 109 parts, among them J1 UJ20-C-H-C-3-SMT-TR, J10 Screw_Terminal_01x02, J11 Screw_Terminal_01x02, J12 Screw_Terminal_01x04, J13 Screw_Terminal_01x02, J14 Screw_Terminal_01x02, J15 Screw_Terminal_01x02, J16 PPPC042LFBN-RC, J17 Screw_Terminal_01x04, J18 Screw_Terminal_01x04, J19 TSW-104-27-G-D, J2 Screw_Terminal_01x04, J20 TSW-104-27-G-D, J3 PPPC042LFBN-RC, J4 Screw_Terminal_01x08, J5 Screw_Terminal_01x08, J6 DM3AT-SF-PEJM5, J7 Screw_Terminal_01x04, J8 Screw_Terminal_01x02, J9 Screw_Terminal_01x04, U1 STM32H757BITx, U10 ADS1115IDGS, U11 ADS1115IDGS, U12 L7805, U2 USBLC6-2SC6, U3 TPS2121RUXR, U4 AP63203QWU-7, U5 ICM-45686, U6 ICM-42688-P, U7 BNO085, U8 XBP9X-DMUS-021, U9 MCP23017T-E_SO

Commit message: fixed schematic issues, started organizing components in PCB
Parts:
- removed Barometer-(U7)1: BMP390L, BMP390L:XDCR_BMP390L
- removed C33: 100uF, Capacitor_SMD:C_1206_3216Metric
- removed C47: 2.2uF, Capacitor_SMD:C_1206_3216Metric
- removed the J4 at (186.7, 69.8)
- removed the J4 at (237.8, 54.0)
- removed the J5 at (186.7, 81.3)
- removed the J5 at (237.8, 65.5)
- removed S1: TL3301NF260QG, TL3301NF260QG:SW_TL3301NF260QG
- added C54: 4.7uF, Capacitor_SMD:C_0805_2012Metric, F.Cu at (131.7, 46.9)
- added C55: 4.7uF, Capacitor_SMD:C_0805_2012Metric, F.Cu at (136.2, 31.8)
- added C56: 4.7uF, Capacitor_SMD:C_0805_2012Metric, F.Cu at (136.2, 34.9)
- added C57: 4.7uF, Capacitor_SMD:C_0805_2012Metric, F.Cu at (136.2, 37.9)
- added C58: 4.7uF, Capacitor_SMD:C_0805_2012Metric, F.Cu at (136.2, 40.9)
- added C59: 100nF, Capacitor_SMD:C_0805_2012Metric, F.Cu at (91.7, 43.9)
- added C60: 1uF, Capacitor_SMD:C_0805_2012Metric, F.Cu at (91.7, 46.9)
- added C61: 4.7uF, Capacitor_SMD:C_0805_2012Metric, F.Cu at (136.2, 43.9)
- added C62: 22uf, Capacitor_SMD:C_0805_2012Metric, F.Cu at (81.4, 161.1)
- added C63: 100nf, Capacitor_SMD:C_0805_2012Metric, F.Cu at (81.4, 164.1)
- added C64: 4.7uf, Capacitor_SMD:C_0805_2012Metric, F.Cu at (81.4, 167.1)
- added C65: 47pf, Capacitor_SMD:C_0805_2012Metric, F.Cu at (81.4, 170.2)
- added C66: 680pf, Capacitor_SMD:C_0805_2012Metric, F.Cu at (81.4, 173.2)
- added C67: 100nf, Capacitor_SMD:C_0805_2012Metric, F.Cu at (85.8, 161.1)
- added C68: 22uf, Capacitor_SMD:C_0805_2012Metric, F.Cu at (85.8, 164.1)
- added C69: 10uF, Capacitor_SMD:C_0805_2012Metric, F.Cu at (85.8, 167.1)
- added C70: 1uF, Capacitor_SMD:C_0805_2012Metric, F.Cu at (85.8, 170.2)
- added C71: 47uF, Capacitor_SMD:C_0805_2012Metric, F.Cu at (85.8, 173.2)
- added D1: GREEN LED, LED_SMD:LED_Cree-PLCC4_5x5mm_CW, F.Cu at (99.3, 163.0)
- added D6: 1N4148W, Diode_SMD:D_SOD-123, F.Cu at (105.6, 168.0)
- added D7: WS2812B-2020, LED_SMD:LED_WS2812B-2020_PLCC4_2.0x2.0mm, F.Cu at (100.9, 156.5)
- added D8: 1N4148W, Diode_SMD:D_SOD-123, F.Cu at (105.6, 171.4)
- added D9: CD4148W, Diode_SMD:D_0805_2012Metric, F.Cu at (131.8, 54.5)
- added J21: XT60-M, XT60-M:AMASS_XT60-M, F.Cu at (89.2, 126.0)
- added J22: Screw_Terminal_01x08, 1984675:PHOENIX_1984675, F.Cu at (130.2, 129.0)
- added J23: Screw_Terminal_01x08, 1984675:PHOENIX_1984675, F.Cu at (130.2, 138.1)
- added J24: Screw_Terminal_01x08, 1984675:PHOENIX_1984675, F.Cu at (130.2, 147.2)
- added J25: Screw_Terminal_01x08, 1984675:PHOENIX_1984675, F.Cu at (130.2, 156.3)
- added J26: Screw_Terminal_01x08, 1984675:PHOENIX_1984675, F.Cu at (80.6, 110.8)
- added J27: Screw_Terminal_01x08, 1984675:PHOENIX_1984675, F.Cu at (80.6, 119.9)
- added J28: Screw_Terminal_01x03, 1984620:PHOENIX_1984620, F.Cu at (40.7, 110.8)
- added J29: Screw_Terminal_01x03, 1984620:PHOENIX_1984620, F.Cu at (40.7, 119.9)
- added J30: Screw_Terminal_01x03, 1984620:PHOENIX_1984620, F.Cu at (40.7, 129.0)
- added J31: Screw_Terminal_01x03, 1984620:PHOENIX_1984620, F.Cu at (40.7, 138.1)
- added J32: Screw_Terminal_01x03, 1984620:PHOENIX_1984620, F.Cu at (40.7, 147.2)
- added J33: Screw_Terminal_01x04, 1984633:PHOENIX_1984633, F.Cu at (113.4, 147.2)
- added J34: Screw_Terminal_01x04, 1984633:PHOENIX_1984633, F.Cu at (113.4, 156.3)
- added J35: Screw_Terminal_01x04, 1984633:PHOENIX_1984633, F.Cu at (113.4, 165.4)
- added J36: PPPC042LFBN-RC, PPPC042LFBN_RC:SULLINS_PPPC042LFBN-RC, F.Cu at (77.8, 97.7)
- added J37: Screw_Terminal_01x03, 1984620:PHOENIX_1984620, F.Cu at (40.7, 156.3)
- added J38: Screw_Terminal_01x03, 1984620:PHOENIX_1984620, F.Cu at (40.7, 165.4)
- added J39: TSW-104-27-G-D, TSW_104_27_G_D:SAMTEC_TSW-104-27-G-D, F.Cu at (81.8, 148.7)
- added J4: Screw_Terminal_01x08, 1984675:PHOENIX_1984675, F.Cu at (130.2, 110.8)
- added J40: Screw_Terminal_01x03, 1984620:PHOENIX_1984620, F.Cu at (40.7, 174.5)
- added J41: STEMMA QT, Connector_JST:JST_SH_SM04B-SRSS-TB_1x04-1MP_P1.00mm_Horizontal, F.Cu at (97.9, 94.2)
- added J42: Screw_Terminal_01x04, 1984633:PHOENIX_1984633, F.Cu at (63.8, 119.9)
- added J43: Screw_Terminal_01x04, 1984633:PHOENIX_1984633, F.Cu at (63.8, 129.0)
- added J44: Screw_Terminal_01x02, 1984617:PHOENIX_1984617, F.Cu at (54.0, 129.0)
- added J45: Screw_Terminal_01x02, 1984617:PHOENIX_1984617, F.Cu at (54.0, 138.1)
- added J46: Screw_Terminal_01x02, 1984617:PHOENIX_1984617, F.Cu at (54.0, 147.2)
- added J47: Screw_Terminal_01x04, 1984633:PHOENIX_1984633, F.Cu at (63.8, 138.1)
- added J48: Screw_Terminal_01x04, 1984633:PHOENIX_1984633, F.Cu at (63.8, 147.2)
- added J49: PPTC032LFBN-RC, Connector_PinSocket_1.00mm:PinSocket_2x03_P1.00mm_Vertical_SMD, F.Cu at (163.0, 163.5)
- added J5: Screw_Terminal_01x08, 1984675:PHOENIX_1984675, F.Cu at (130.2, 119.9)
- added J50: PCB.RPSMAFRA.HT, KiCad(1):PCBRPSMAFRAHT, F.Cu at (102.9, 73.6)
- added J52: PPTC041LFBN-RC, Connector_PinSocket_2.54mm:PinSocket_1x04_P2.54mm_Vertical, F.Cu at (161.8, 150.8)
- added LS1: CMT-7525-80-SMT-TR, CMT_7525_80_SMT_TR:XDCR_CMT-7525-80-SMT-TR, F.Cu at (120.4, 64.9)
- added Q1: AO3400A, Package_TO_SOT_SMD:SOT-23, F.Cu at (81.6, 152.9)
- added Q2: AO3400A, Package_TO_SOT_SMD:SOT-23, F.Cu at (81.6, 157.4)
- added Q3: AO3401A, Package_TO_SOT_SMD:SOT-23, F.Cu at (86.5, 152.9)
- added Q4: AO3401A, Package_TO_SOT_SMD:SOT-23, F.Cu at (86.5, 157.4)
- added Q5: AO3400A, Package_TO_SOT_SMD:SOT-23, F.Cu at (91.4, 152.9)
- added Q6: AO3400A, Package_TO_SOT_SMD:SOT-23, F.Cu at (91.4, 157.4)
- added Q7: AO3401A, Package_TO_SOT_SMD:SOT-23, F.Cu at (96.3, 152.9)
- added Q8: AO3401A, Package_TO_SOT_SMD:SOT-23, F.Cu at (96.3, 157.4)
- added Q9: FMMT619TA, KiCad3:SOT95P237X112-3N, F.Cu at (132.0, 50.7)
- added R17: 1.3k, Resistor_SMD:R_0805_2012Metric, F.Cu at (93.6, 132.3)
- added R18: 10k, Resistor_SMD:R_0805_2012Metric, F.Cu at (82.7, 67.8)
- added R19: 23.7k, Resistor_SMD:R_0805_2012Metric, F.Cu at (93.6, 135.2)
- added R20: 374k, Resistor_SMD:R_0805_2012Metric, F.Cu at (93.6, 138.2)
- added R21: 10k, Resistor_SMD:R_0805_2012Metric, F.Cu at (82.7, 70.8)
- added R22: 100k, Resistor_SMD:R_0805_2012Metric, F.Cu at (93.6, 141.2)
- added R23: 1.07M, Resistor_SMD:R_0805_2012Metric, F.Cu at (93.6, 144.1)
- added R24: 120k, Resistor_SMD:R_0805_2012Metric, F.Cu at (93.6, 147.1)
- added R25: 10k, Resistor_SMD:R_0805_2012Metric, F.Cu at (98.0, 132.3)
- added R26: 10k, Resistor_SMD:R_0805_2012Metric, F.Cu at (98.0, 135.2)
- added R27: 1k, Resistor_SMD:R_0805_2012Metric, F.Cu at (98.0, 138.2)
- added R28: 1k, Resistor_SMD:R_0805_2012Metric, F.Cu at (98.0, 141.2)
- added R29: 1k, Resistor_SMD:R_0805_2012Metric, F.Cu at (98.0, 144.1)
- added R30: 1k, Resistor_SMD:R_0805_2012Metric, F.Cu at (98.0, 147.1)
- added R31: 10k, Resistor_SMD:R_0805_2012Metric, F.Cu at (102.4, 132.3)
- added R32: 10k, Resistor_SMD:R_0805_2012Metric, F.Cu at (102.4, 135.2)
- added R33: 1k, Resistor_SMD:R_0805_2012Metric, F.Cu at (102.4, 138.2)
- added R34: 1k, Resistor_SMD:R_0805_2012Metric, F.Cu at (102.4, 141.2)
- added R35: 10k, Resistor_SMD:R_0805_2012Metric, F.Cu at (82.7, 73.7)
- added R36: 10k, Resistor_SMD:R_0805_2012Metric, F.Cu at (82.7, 76.7)
- added R37: 10k, Resistor_SMD:R_0805_2012Metric, F.Cu at (82.7, 79.6)
- added R38: 5k, Resistor_SMD:R_0805_2012Metric, F.Cu at (102.4, 144.1)
- added R39: 5k, Resistor_SMD:R_0805_2012Metric, F.Cu at (102.4, 147.1)
- added R40: 5k, Resistor_SMD:R_0805_2012Metric, F.Cu at (106.8, 132.3)
- added R41: 5k, Resistor_SMD:R_0805_2012Metric, F.Cu at (106.8, 135.2)
- added R42: 5k, Resistor_SMD:R_0805_2012Metric, F.Cu at (106.8, 138.2)
- added R43: 5k, Resistor_SMD:R_0805_2012Metric, F.Cu at (106.8, 141.2)
- added R44: 5k, Resistor_SMD:R_0805_2012Metric, F.Cu at (106.8, 144.1)
- added R45: 180, Resistor_SMD:R_0805_2012Metric, F.Cu at (136.2, 54.5)
- added U14: MS5611-01BA, Package_LGA:LGA-8_3x5mm_P1.25mm, F.Cu at (68.2, 66.3)
- added U15: TPS7A4701xRGW, Package_DFN_QFN:Texas_RGW0020A_VQFN-20-1EP_5x5mm_P0.65mm_EP3.15x3.15mm, F.Cu at (125.9, 41.3)
- added U17: MCP1826ST-3302E/DB, footprints8:SOT-223_3MC_MCH-L, F.Cu at (117.7, 35.0)
- added U18: MCP1826ST-3302E/DB, footprints8:SOT-223_3MC_MCH-L, F.Cu at (117.7, 44.2)
- added U19: MCP1826ST-3302E/DB, footprints8:SOT-223_3MC_MCH-L, F.Cu at (117.7, 53.5)
- added U20: TPS7A4701xRGW, Package_DFN_QFN:Texas_RGW0020A_VQFN-20-1EP_5x5mm_P0.65mm_EP3.15x3.15mm, F.Cu at (125.9, 48.6)
- added U21: TPS61089, Package_DFN_QFN:Texas_VQFN-RNR0011A-11, F.Cu at (101.0, 152.8)
- added U22: TPS7A4701xRGW, Package_DFN_QFN:Texas_RGW0020A_VQFN-20-1EP_5x5mm_P0.65mm_EP3.15x3.15mm, F.Cu at (99.0, 170.0)
- C1, C10, C11, C12, C13, C14, C15, C16, C17, C18, C19, C2, C20, C21, C22, C23, C24, C25, C27, C28, C3, C30, C34, C36, C37, C38, C39, C4, C40, C43, C46, C48, C49, C5, C6, C7, C8, C9: footprint Capacitor_SMD:C_1206_3216Metric -> Capacitor_SMD:C_0805_2012Metric
- C26: value 100nF -> 1uF; footprint Capacitor_SMD:C_1206_3216Metric -> Capacitor_SMD:C_0805_2012Metric
- C29: value 0.01uF -> 10nF; footprint Capacitor_SMD:C_1206_3216Metric -> Capacitor_SMD:C_0805_2012Metric
- C31: value 22uF -> 1uF; footprint Capacitor_SMD:C_1206_3216Metric -> Capacitor_SMD:C_0805_2012Metric
- C32: value 22uF -> 47uF; footprint Capacitor_SMD:C_1206_3216Metric -> Capacitor_SMD:C_0805_2012Metric
- C35: value 100nF -> 2.2uF ESR<100mohm; footprint Capacitor_SMD:C_1206_3216Metric -> Capacitor_SMD:C_0805_2012Metric
- C41, C42: value 2.2uF -> 2.2uF ESR<100mohm; footprint Capacitor_SMD:C_1206_3216Metric -> Capacitor_SMD:C_0805_2012Metric
- C44: value 10nF -> 2.2uF; footprint Capacitor_SMD:C_1206_3216Metric -> Capacitor_SMD:C_0805_2012Metric
- C45: value 2.2uF -> 10nF; footprint Capacitor_SMD:C_1206_3216Metric -> Capacitor_SMD:C_0805_2012Metric
- C51: value 0.33uF -> 10uF; footprint Capacitor_SMD:C_1206_3216Metric -> Capacitor_SMD:C_0805_2012Metric
- C52: value 100nF -> 10uF; footprint Capacitor_SMD:C_1206_3216Metric -> Capacitor_SMD:C_0805_2012Metric
- D2: value LED -> BLUE LED
- D3: value LED -> RED LED
- D4: value LED -> GREEN LED
- J10, J11, J13, J14, J15, J8: footprint footprints5:CONN_1729128_PXC -> 1984617:PHOENIX_1984617
- J12, J18, J2, J7, J9: footprint footprints6:CONN_1715747_PXC -> 1984633:PHOENIX_1984633
- J17: value Screw_Terminal_01x04 -> Screw_Terminal_01x02; footprint footprints6:CONN_1715747_PXC -> 1984617:PHOENIX_1984617
- L1: value 3.3uH -> 2.2uH; footprint Inductor_SMD:L_1206_3216Metric -> Inductor_SMD:L_0805_2012Metric
- R1, R2: value 5k1 -> 5k; footprint Resistor_SMD:R_1206_3216Metric -> Resistor_SMD:R_0805_2012Metric
- R10, R9: value 2.2kR -> 2.2k; footprint Resistor_SMD:R_1206_3216Metric -> Resistor_SMD:R_0805_2012Metric
- R11, R12, R14, R8: value 10kR -> 10k; footprint Resistor_SMD:R_1206_3216Metric -> Resistor_SMD:R_0805_2012Metric
- R13: value 82R -> 4.7kR; footprint Resistor_SMD:R_1206_3216Metric -> Resistor_SMD:R_0805_2012Metric
- R15: value 50R -> 620R; footprint Resistor_SMD:R_1206_3216Metric -> Resistor_SMD:R_0805_2012Metric
- R16: value 270R -> 1.3kR; footprint Resistor_SMD:R_1206_3216Metric -> Resistor_SMD:R_0805_2012Metric
- R3: value 22k1 -> 22k; footprint Resistor_SMD:R_1206_3216Metric -> Resistor_SMD:R_0805_2012Metric
- R4: value 41k2 -> 41.2k; footprint Resistor_SMD:R_1206_3216Metric -> Resistor_SMD:R_0805_2012Metric
- R5, R7: value 5kR -> 5k; footprint Resistor_SMD:R_1206_3216Metric -> Resistor_SMD:R_0805_2012Metric
- R6: value 23k7 -> 23k; footprint Resistor_SMD:R_1206_3216Metric -> Resistor_SMD:R_0805_2012Metric
- U12: value L7805 -> XBP9X-DMRS-001; footprint L7805:TO255P1020X450X2000-3 -> XBP9X_DMUS_021:XCVR_XBP9X-DMUS-021
- U4: value AP63203QWU-7 -> TPS7A4701xRGW; footprint footprints2:TSOT26_DIO -> Package_DFN_QFN:Texas_RGW0020A_VQFN-20-1EP_5x5mm_P0.65mm_EP3.15x3.15mm
- U8: value XBP9X-DMUS-021 -> ADS1115IDGS; footprint XBP9X-DMUS-021:DIP2200W51P200L3294H279Q20P -> Package_SO:TSSOP-10_3x3mm_P0.5mm
- moved U12 220.4 mm to (45.0, 83.0)
- moved D5 194.0 mm to (67.9, 87.2)
- moved U10 193.9 mm to (91.5, 166.6)
- moved U11 193.9 mm to (91.5, 171.2)
- moved C50 187.9 mm to (68.6, 83.8)
- moved J17 185.0 mm to (54.0, 119.9)
- moved J19 182.1 mm to (81.8, 135.4)
- moved J20 182.1 mm to (81.8, 142.0)
- moved R13 178.2 mm to (78.3, 76.7)
- moved R16 175.4 mm to (82.7, 64.9)
- moved R15 175.3 mm to (82.7, 61.9)
- moved J18 174.0 mm to (63.8, 110.8)
- moved J16 169.4 mm to (77.8, 91.0)
- moved J3 169.4 mm to (77.8, 84.4)
- moved C49 168.4 mm to (91.7, 40.9)
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Connections:
- net /Chips/SD_CLK renamed SD_CLK
- net /Chips/SD_CMD renamed SD_CMD
- net /Chips/SD_DAT0 renamed SD_DAT0
- net /Chips/SD_DAT1 renamed SD_DAT1
- net /Chips/SD_DAT2 renamed SD_DAT2
- net /Chips/SD_DAT3 renamed SD_DAT3
- net Net-(U1-BOOT0) renamed BOOT
- net Net-(U1-VCAPDSI) renamed VCAPDSI
- C1 pad 1: GND -> 3V3_MCU
- C1 pad 2: 3V3 -> VDDSMPS
- C10 pad 1: GND -> 3V3_MCU
- C10 pad 2: 3V3 -> VDDSMPS
- C11 pad 1: GND -> 3V3_MCU
- C11 pad 2: 3V3 -> VDDSMPS
- C12 pad 1: GND -> 3V3_MCU
- C12 pad 2: 3V3 -> VDDSMPS
- C13 pad 1: GND -> 3V3_MCU
- C13 pad 2: 3V3 -> VDDSMPS
- C14 pad 1: GND -> 3V3_MCU
- C14 pad 2: 3V3 -> VDDSMPS
- C15 pad 1: GND -> 3V3_MCU
- C15 pad 2: 3V3 -> VDDSMPS
- C16 pad 1: GND -> 3V3_MCU
- C16 pad 2: 3V3 -> VDDSMPS
- C17 pad 1: GND -> 3V3_MCU
- C17 pad 2: 3V3 -> VDDSMPS
- C18 pad 1: GND -> 3V3_MCU
- C18 pad 2: 3V3 -> VDDSMPS
- C19 pad 1: GND -> 3V3_MCU
- C19 pad 2: 3V3 -> VDDSMPS
- C2 pad 1: GND -> 3V3_MCU
- C2 pad 2: 3V3 -> VDDSMPS
- C20 pad 1: GND -> 3V3_MCU
- C20 pad 2: 3V3 -> VDDSMPS
- C21 pad 1: GND -> 3V3_MCU
- C21 pad 2: 3V3 -> VDDSMPS
- C22 pad 1: GND -> 3V3
- C22 pad 2: 3V3 -> VDDSMPS
- C23 pad 1: GND -> 3V3
- C23 pad 2: 3V3 -> VDDSMPS
- C24 pad 1: GND -> 3V3
- C24 pad 2: 3V3 -> VDDSMPS
- C25 pad 1: GND -> 3V3_MCU
- C25 pad 2: USB_VBUS -> VDDSMPS
- C26 pad 1: GND -> 3V3_MCU
- C26 pad 2: 3V3 -> VDDSMPS
- C27 pad 1: Net-(C27-Pad1) -> USB_VBUS
- C27 pad 2: GND -> VDDSMPS
- C28 pad 2: GND -> VDDSMPS
- C29 pad 2: GND -> VDDSMPS
- C3 pad 1: GND -> 3V3_MCU
- C3 pad 2: 3V3 -> VDDSMPS
- C30 pad 1: GND -> V_OUT
- C30 pad 2: V_OUT -> VDDSMPS
- C31 pad 1: GND -> unconnected-(C31-Pad1)
- C31 pad 2: Net-(C31-Pad2) -> VDDSMPS
- C32 pad 1: Net-(C31-Pad2) -> /Chips/Regulators/5V_XB
- C32 pad 2: 3V3 -> VDDSMPS
- C34 pad 1: GND -> 3V3_MCU
- C34 pad 2: 3V3 -> VDDSMPS
- C35 pad 1: GND -> VDDSMPS
- C35 pad 2: 3V3 -> VCAP
- C36 pad 1: 3V3 -> 3V3_SENS
- C36 pad 2: GND -> VDDSMPS
- C37 pad 1: 3V3 -> 3V3_SENS
- C37 pad 2: GND -> VDDSMPS
- C38 pad 1: GND -> VDDSMPS
- C38 pad 2: 3V3 -> 3V3_SENS
- C39 pad 1: GND -> VDDSMPS
- C39 pad 2: 3V3 -> 3V3_SENS
- C4 pad 1: GND -> 3V3_MCU
- C4 pad 2: 3V3 -> VDDSMPS
- C40 pad 2: GND -> VDDSMPS
- C41 pad 1: GND -> VDDSMPS
- C41 pad 2: Net-(C41-Pad2) -> VCAP
- C42 pad 1: GND -> VDDSMPS
- C42 pad 2: Net-(C42-Pad2) -> VCAP
- C43 pad 1: GND -> VDDSMPS
- C43 pad 2: 3V3 -> 3V3_SENS
- C44 pad 1: 3V3 -> VDDSMPS
- C44 pad 2: GND -> 3V3_SENS
- C45 pad 1: GND -> 3V3_SENS
- C45 pad 2: 3V3 -> VDDSMPS
- C46 pad 1: GND -> VDDSMPS
- C46 pad 2: 3V3 -> 3V3_SENS
- C48 pad 1: GND -> VDDSMPS
- C48 pad 2: 3V3 -> 3V3_XB
- C49 pad 1: GND -> VDDSMPS
- C49 pad 2: 3V3 -> 3V3_XB
- C5 pad 1: GND -> 3V3_MCU
- C5 pad 2: 3V3 -> VDDSMPS
- C50 pad 1: GND -> VDDSMPS
- C50 pad 2: 3V3 -> 3V3_XB
- C51 pad 1: 7.4V -> V_OUT
- C51 pad 2: GND -> VDDSMPS
- C52 pad 1: 5V -> V_OUT
- C52 pad 2: GND -> VDDSMPS
- C6 pad 1: GND -> 3V3_MCU
- C6 pad 2: 3V3 -> VDDSMPS
- C7 pad 1: GND -> 3V3_MCU
- C7 pad 2: 3V3 -> VDDSMPS
- C8 pad 1: GND -> 3V3_MCU
- C8 pad 2: 3V3 -> VDDSMPS
- C9 pad 1: GND -> 3V3_MCU
- C9 pad 2: 3V3 -> VDDSMPS
- D2 pad 1: USB_VBUS -> VDDSMPS
- D3 pad 1: GND -> VDDSMPS
- D4 pad 1: Net-(D4-K) -> VDDSMPS
- D5 pad 2: GND -> VDDSMPS
- D5 pad 4: 3V3 -> 3V3_MCU
- J1 pad A12_B1: GND -> VDDSMPS
- J1 pad A1_B12: GND -> VDDSMPS
- J1 pad A4_B9: Net-(C27-Pad1) -> USB_VBUS
- J1 pad A9_B4: Net-(C27-Pad1) -> USB_VBUS
- J1 pad SH1: GND -> VDDSMPS
- J1 pad SH2: GND -> VDDSMPS
- J1 pad SH3: GND -> VDDSMPS
- J1 pad SH4: GND -> VDDSMPS
- J12 pad 1: GND -> VDDSMPS
- J12 pad 2: GND -> VDDSMPS
- J12 pad 3: GND -> VDDSMPS
- J12 pad 4: GND -> VDDSMPS
- J16 pad 2: HDR_GPIO1 -> SERVO1
- J16 pad 3: HDR_GPIO2 -> SERVO2
- J16 pad 4: HDR_GPIO3 -> SERVO3
- J16 pad 5: HDR_GPIO4 -> SERVO4
- J16 pad 6: HDR_GPIO5 -> SERVO5
- J16 pad 7: HDR_GPIO6 -> SERVO6
- J16 pad 8: HDR_GPIO7 -> SERVO7
- J17 pad 1: ADC1_IN0 -> ADC1_IN2
- J17 pad 2: ADC1_IN1 -> ADC1_IN3
- J19 pad 01: HDR_GPIO8 -> PYRO1_GPIO
- J19 pad 05: ADC2_SDA -> TEMP_SCL
- J19 pad 06: ADC2_SCL -> TEMP_SCL
- J19 pad 07: PYRO2 -> PYRO2_GPIO
- J19 pad 08: GND -> VDDSMPS
- J20 pad 02: HDR_GPIO1 -> SERVO1
- J20 pad 03: HDR_GPIO2 -> SERVO2
- J20 pad 04: HDR_GPIO3 -> SERVO3
- J20 pad 05: HDR_GPIO4 -> SERVO4
- J20 pad 06: HDR_GPIO5 -> SERVO5
- J20 pad 07: HDR_GPIO6 -> SERVO6
- J20 pad 08: HDR_GPIO7 -> SERVO7
- J3 pad 1: HDR_GPIO8 -> PYRO1_GPIO
- J3 pad 5: ADC2_SDA -> TEMP_SCL
- J3 pad 6: ADC2_SCL -> TEMP_SCL
- J3 pad 7: PYRO2 -> PYRO2_GPIO
- J3 pad 8: GND -> VDDSMPS
- J6 pad 4: 3V3 -> 3V3_SENS
- J6 pad 6: GND -> VDDSMPS
- J6 pad P1: GND -> VDDSMPS
- J6 pad P2: GND -> VDDSMPS
- J6 pad P3: GND -> VDDSMPS
- J6 pad P4: GND -> VDDSMPS
- J8 pad 1: UART5_RX -> HDR_GPIO1
- J8 pad 2: UART5_TX -> HDR_GPIO3
- J9 pad 1: 3.3V -> 3V3
- J9 pad 2: 5V -> USB_VBUS
- J9 pad 3: 5V -> USB_VBUS
- J9 pad 4: 5V -> USB_VBUS
- L1 pad 1: Net-(U4-SW) -> 7.4V
- L1 pad 2: 3V3 -> Net-(U21-SW)
- R1 pad 2: GND -> VDDSMPS
- R10 pad 2: 3V3 -> 3V3_SENS
- R11 pad 1: 3V3 -> BNO_CS
- R11 pad 2: ICM456_CS -> 3V3
- R12 pad 1: 3V3 -> 3V3_SENS
- R12 pad 2: ICM426_CS -> BNO_NRST
- R13 pad 2: Net-(C27-Pad1) -> USB_VBUS
- R14 pad 2: Net-(R14-Pad2) -> VDDSMPS
- R15 pad 1: Net-(D3-A) -> Net-(U12-DIO1/AD1)
- R15 pad 2: Net-(U8-DIO10/PWM0) -> Net-(D3-A)
- R2 pad 2: GND -> VDDSMPS
- R3 pad 2: GND -> VDDSMPS
- R4 pad 1: Net-(D4-K) -> 7.4V
- R5 pad 2: GND -> VDDSMPS
- R7 pad 2: GND -> VDDSMPS
- R9 pad 2: 3V3 -> 3V3_SENS
- U1 pad 100: 3V3 -> 3V3_MCU
- U1 pad 101: UART5_RX -> SLN_1
- U1 pad 102: UART5_TX -> HDR_GPIO2
- U1 pad 103: unconnected-(U1-PB14-Pad103) -> HDR_GPIO1
- U1 pad 104: unconnected-(U1-PB15-Pad104) -> PYRO1_CONT
- U1 pad 105: HDR_GPIO1 -> unconnected-(U1-PD8-Pad105)
- U1 pad 106: HDR_GPIO2 -> unconnected-(U1-PD9-Pad106)
- U1 pad 107: HDR_GPIO3 -> SLN_2
- U1 pad 108: 3V3 -> 3V3_MCU
- U1 pad 109: GND -> VDDSMPS
- U1 pad 110: HDR_GPIO4 -> SPKG
- U1 pad 111: HDR_GPIO5 -> HDR_GPIO3
- U1 pad 112: HDR_GPIO6 -> PYRO2_CONT
- U1 pad 113: GND -> VDDSMPS
- U1 pad 114: 3V3 -> 3V3_MCU
- U1 pad 115: HDR_GPIO7 -> PYRO1_GPIO
- U1 pad 116: HDR_GPIO8 -> PYRO2_GPIO
- U1 pad 117: 3V3 -> 3V3_MCU
- U1 pad 118: GND -> VDDSMPS
- U1 pad 123: GND -> VDDSMPS
- U1 pad 129: GND -> VDDSMPS
- U1 pad 13: XB_TX -> unconnected-(U1-PI9-Pad13)
- U1 pad 130: unconnected-(U1-PG2-Pad130) -> SERVO7
- U1 pad 131: unconnected-(U1-PG3-Pad131) -> SERVO6
- U1 pad 132: GND -> VDDSMPS
- U1 pad 133: 3V3 -> 3V3_MCU
- U1 pad 134: unconnected-(U1-PG4-Pad134) -> SERVO5
- U1 pad 135: unconnected-(U1-PG5-Pad135) -> SERVO4
- U1 pad 136: unconnected-(U1-PG6-Pad136) -> SERVO3
- U1 pad 137: unconnected-(U1-PG7-Pad137) -> SERVO2
- U1 pad 138: unconnected-(U1-PG8-Pad138) -> SERVO1
- U1 pad 139: GND -> VDDSMPS
- U1 pad 140: USB_VBUS -> 3V3_MCU
- U1 pad 141: 3V3 -> 3V3_MCU
- U1 pad 149: unconnected-(U1-PA11-Pad149) -> USB_D-
- U1 pad 150: unconnected-(U1-PA12-Pad150) -> USB_D+
- U1 pad 151: unconnected-(U1-PA13-Pad151) -> DEBUG_SWDIO
- U1 pad 152: Net-(C42-Pad2) -> VCAP
- U1 pad 153: GND -> VDDSMPS
- U1 pad 155: 3V3 -> 3V3_MCU
- U1 pad 156: unconnected-(U1-PH13-Pad156) -> BNO_CLKSEL0
- U1 pad 157: unconnected-(U1-PH14-Pad157) -> BARO_CS
- U1 pad 158: unconnected-(U1-PH15-Pad158) -> BNO_CS
- U1 pad 159: unconnected-(U1-PI0-Pad159) -> BNO_WAKE/PS0
- U1 pad 16: GND -> VDDSMPS
- U1 pad 160: GND -> VDDSMPS
- U1 pad 161: 3V3 -> 3V3_MCU
- U1 pad 162: unconnected-(U1-PI1-Pad162) -> BNO_NRST
- U1 pad 163: unconnected-(U1-PI2-Pad163) -> BNO_BOOTN
- U1 pad 165: unconnected-(U1-PA14-Pad165) -> DEBUG_SWCLK
- U1 pad 17: 3V3 -> 3V3_MCU
- U1 pad 177: unconnected-(U1-PD7-Pad177) -> ICM456_MOSI
- U1 pad 178: GND -> VDDSMPS
- U1 pad 179: 3V3 -> 3V3_MCU
- U1 pad 18: GND -> VDDSMPS
- U1 pad 180: unconnected-(U1-PG9-Pad180) -> ICM456_MISO
- U1 pad 182: unconnected-(U1-PG11-Pad182) -> ICM456_CLK
- U1 pad 184: SPI6_CLK -> unconnected-(U1-PG13-Pad184)
- U1 pad 186: GND -> VDDSMPS
- U1 pad 187: 3V3 -> 3V3_MCU
- U1 pad 191: unconnected-(U1-PB5-Pad191) -> XB_RX
- U1 pad 192: EXP_SCL -> XB_TX
- U1 pad 195: unconnected-(U1-PB8-Pad195) -> EXP_SCL
- U1 pad 199: Net-(C47-Pad2) -> VCAP
- U1 pad 20: GND -> VDDSMPS
- U1 pad 200: GND -> VDDSMPS
- U1 pad 201: 3V3 -> 3V3_MCU
- U1 pad 207: GND -> VDDSMPS
- U1 pad 208: 3V3 -> 3V3_MCU
- U1 pad 21: GND -> VDDSMPS
- U1 pad 24: unconnected-(U1-PF2-Pad24) -> MISC_GPIO4
- U1 pad 25: unconnected-(U1-PF3-Pad25) -> MISC_GPIO3
- U1 pad 26: unconnected-(U1-PF4-Pad26) -> MISC_GPIO2
- U1 pad 27: unconnected-(U1-PF5-Pad27) -> MISC_GPIO1
- U1 pad 28: GND -> VDDSMPS
- U1 pad 29: 3V3 -> 3V3_MCU
- U1 pad 3: unconnected-(U1-PE4-Pad3) -> XB_RESET
- U1 pad 32: SPI6_MISO -> SPI5_MISO
- U1 pad 37: unconnected-(U1-NRST-Pad37) -> RST
- U1 pad 42: GND -> VDDSMPS
- U1 pad 43: 3V3 -> 3V3_MCU
- U1 pad 44: 3V3 -> 3V3_MCU
- U1 pad 45: XB_RX -> unconnected-(U1-PA0-Pad45)
- U1 pad 49: 3V3 -> 3V3_MCU
- U1 pad 50: GND -> VDDSMPS
- U1 pad 55: GND -> VDDSMPS
- U1 pad 56: 3V3 -> 3V3_MCU
- U1 pad 57: unconnected-(U1-PA4-Pad57) -> BUZZ
- U1 pad 58: ICM456_CLK -> SPI6_CLK
- U1 pad 59: ICM456_MISO -> unconnected-(U1-PA6-Pad59)
- U1 pad 6: GND -> VDDSMPS
- U1 pad 60: ICM456_MOSI -> unconnected-(U1-PA7-Pad60)
- U1 pad 61: unconnected-(U1-PC4-Pad61) -> ICM426_INT1
- U1 pad 63: unconnected-(U1-PB0-Pad63) -> MCP230_INT1
- U1 pad 64: unconnected-(U1-PB1-Pad64) -> MCP230_INT2
- U1 pad 66: unconnected-(U1-PI15-Pad66) -> EXP_SDA
- U1 pad 67: unconnected-(U1-PF11-Pad67) -> ICM456_INT
- U1 pad 69: unconnected-(U1-PF13-Pad69) -> BNO_INT
- U1 pad 7: 3V3 -> 3V3_MCU
- U1 pad 73: GND -> VDDSMPS
- U1 pad 74: 3V3 -> 3V3_MCU
- U1 pad 75: unconnected-(U1-PG1-Pad75) -> XB_INT
- U1 pad 78: unconnected-(U1-PE9-Pad78) -> ICM456_INT2
- U1 pad 79: GND -> VDDSMPS
- U1 pad 8: 3V3 -> 3V3_MCU
- U1 pad 80: 3V3 -> 3V3_MCU
- U1 pad 81: unconnected-(U1-PE10-Pad81) -> STM_CSN
- U1 pad 82: unconnected-(U1-PE11-Pad82) -> BARO_CS
- U1 pad 83: unconnected-(U1-PE12-Pad83) -> ICM426_INT2
- U1 pad 84: unconnected-(U1-PE13-Pad84) -> XBP_CS
- U1 pad 85: unconnected-(U1-PE14-Pad85) -> ICM406_CS
- U1 pad 86: unconnected-(U1-PE15-Pad86) -> SPI5_CS
- U1 pad 88: unconnected-(U1-PB11-Pad88) -> SPI6_CS
- U1 pad 89: Net-(C41-Pad2) -> VCAP
- U1 pad 90: GND -> VDDSMPS
- U1 pad 93: ADC2_SCL -> TEMP_SCL
- U1 pad 94: ADC2_SDA -> TEMP_SCL
- U1 pad 99: GND -> VDDSMPS
- U10 pad 1: unconnected-(U10-ADDR-Pad1) -> VDDSMPS
- U10 pad 3: GND -> VDDSMPS
- U10 pad 4: ADC1_IN0 -> PYRO1_CONT_READ
- U10 pad 5: ADC1_IN1 -> PYRO2_CONT_READ
- U10 pad 8: 5V -> USB_VBUS
- U11 pad 1: unconnected-(U11-ADDR-Pad1) -> ADC2_SDA
- U11 pad 10: ADC2_SDA -> ADC2_SCL
- U11 pad 3: GND -> VDDSMPS
- U11 pad 8: 5V -> USB_VBUS
- U11 pad 9: ADC2_SCL -> ADC2_SDA
- U12 pad 1: 7.4V -> (no net)
- U12 pad 2: GND -> 3V3_XB
- U12 pad 3: 5V -> XB_TX
- U2 pad 2: GND -> VDDSMPS
- U2 pad 5: Net-(C27-Pad1) -> USB_VBUS
- U3 pad 12: GND -> VDDSMPS
- U3 pad 2: Net-(D4-K) -> 7.4V
- U3 pad 3: GND -> VDDSMPS
- U3 pad 6: GND -> VDDSMPS
- U3 pad 9: GND -> VDDSMPS
- U4 pad 1: 3V3 -> /Chips/Regulators/5V_SENS
- U4 pad 2: V_OUT -> (no net)
- U4 pad 3: V_OUT -> unconnected-(U4-SENSE/FB-Pad3)
- U4 pad 4: GND -> unconnected-(U4-6.4V-Pad4)
- U4 pad 5: Net-(U4-SW) -> unconnected-(U4-6.4V-Pad5)
- U4 pad 6: Net-(U4-BST) -> VDDSMPS
- U5 pad 10: unconnected-(U5-RESV/AUX1_CS-Pad10) -> VDDSMPS
- U5 pad 11: unconnected-(U5-RESV/AUX1_SDO-Pad11) -> VDDSMPS
- U5 pad 12: ICM456_CS -> VDDSMPS
- U5 pad 2: unconnected-(U5-RESV/AUX1_SDIO/AUX1_SDI/MAS_DA-Pad2) -> VDDSMPS
- U5 pad 3: unconnected-(U5-RESV/AUX1_SCLK/MAS_CLK-Pad3) -> VDDSMPS
- U5 pad 5: 3V3 -> 3V3_SENS
- U5 pad 6: GND -> VDDSMPS
- U5 pad 7: unconnected-(U5-RESV-Pad7) -> VDDSMPS
- U5 pad 8: 3V3 -> 3V3_SENS
- U5 pad 9: unconnected-(U5-INT2/FSYNC/CLKIN-Pad9) -> ICM456_INT2
- U6 pad 10: unconnected-(U6-RESV_10-Pad10) -> VDDSMPS
- U6 pad 11: GND -> VDDSMPS
- U6 pad 12: ICM426_CS -> VDDSMPS
- U6 pad 2: unconnected-(U6-RESV_2-Pad2) -> VDDSMPS
- U6 pad 3: unconnected-(U6-RESV_3-Pad3) -> VDDSMPS
- U6 pad 4: ICM426_INT -> ICM426_INT1
- U6 pad 5: 3V3 -> 3V3_SENS
- U6 pad 6: GND -> VDDSMPS
- U6 pad 7: unconnected-(U6-RESV_7-Pad7) -> VDDSMPS
- U6 pad 8: 3V3 -> 3V3_SENS
- U6 pad 9: unconnected-(U6-INT2/FSYNC/CLKIN-Pad9) -> ICM426_INT2
- U7 pad 14: STM_INTN -> BNO_INT
- U7 pad 18: STM_CSN -> BNO_CS
- U7 pad 2: GND -> VDDSMPS
- U7 pad 25: GND -> VDDSMPS
- U7 pad 28: 3V3 -> 3V3_SENS
- U7 pad 3: 3V3 -> 3V3_SENS
- U7 pad 5: 3V3 -> 3V3_SENS
- U8 pad 1: 3V3 -> USB_VBUS
- U8 pad 10: GND -> ADC3_SCL
- U8 pad 2: XB_TX -> unconnected-(U8-ALERT/RDY-Pad2)
- U8 pad 3: XB_RX -> VDDSMPS
- U8 pad 4: B/R_MISO -> ADC3_IN0
- U8 pad 5: unconnected-(U8-~{RESET}-Pad5) -> ADC3_IN1
- U8 pad 6: Net-(U8-DIO10/PWM0) -> ADC3_IN2
- U8 pad 7: unconnected-(U8-DIO11/PWM1-Pad7) -> ADC3_IN3
- U8 pad 8: (no net) -> USB_VBUS
- U8 pad 9: unconnected-(U8-NDTR/SLEEP_RQ/DIO8-Pad9) -> ADC3_SDA
- U9 pad 10: GND -> VDDSMPS
- U9 pad 15: unconnected-(U9-A0-Pad15) -> VDDSMPS
- U9 pad 16: unconnected-(U9-A1-Pad16) -> VDDSMPS
- U9 pad 17: unconnected-(U9-A2-Pad17) -> VDDSMPS
- U9 pad 18: unconnected-(U9-~{RESET}-Pad18) -> EXP_SDA
- U9 pad 19: unconnected-(U9-INTB-Pad19) -> MCP230_INT1
- U9 pad 20: unconnected-(U9-INTA-Pad20) -> MCP230_INT2
- U9 pad 9: 5V -> 3V3_SENS

Commit message: layout and changed screw term size
Parts:
- removed C62, C68: 22uf, Capacitor_SMD:C_0805_2012Metric
- removed C63, C67: 100nf, Capacitor_SMD:C_0805_2012Metric
- removed C64: 4.7uf, Capacitor_SMD:C_0805_2012Metric
- removed C65: 47pf, Capacitor_SMD:C_0805_2012Metric
- removed C66: 680pf, Capacitor_SMD:C_0805_2012Metric
- removed C69: 10uF, Capacitor_SMD:C_0805_2012Metric
- removed C70: 1uF, Capacitor_SMD:C_0805_2012Metric
- removed C71: 47uF, Capacitor_SMD:C_0805_2012Metric
- removed D1: GREEN LED, LED_SMD:LED_Cree-PLCC4_5x5mm_CW
- removed D6, D8: 1N4148W, Diode_SMD:D_SOD-123
- removed D7: WS2812B-2020, LED_SMD:LED_WS2812B-2020_PLCC4_2.0x2.0mm
- removed J17, J44, J45, J46, J8: Screw_Terminal_01x02, 1984617:PHOENIX_1984617
- removed J18, J42, J43, J47, J48: Screw_Terminal_01x04, 1984633:PHOENIX_1984633
- removed J19, J20, J39: TSW-104-27-G-D, TSW_104_27_G_D:SAMTEC_TSW-104-27-G-D
- removed J21: XT60-M, XT60-M:AMASS_XT60-M
- removed J26, J27: Screw_Terminal_01x08, 1984675:PHOENIX_1984675
- removed J28, J29, J30, J31, J32, J37, J38, J40: Screw_Terminal_01x03, 1984620:PHOENIX_1984620
- removed L1: 2.2uH, Inductor_SMD:L_0805_2012Metric
- removed Q1, Q2, Q5, Q6: AO3400A, Package_TO_SOT_SMD:SOT-23
- removed Q3, Q4, Q7, Q8: AO3401A, Package_TO_SOT_SMD:SOT-23
- removed R17: 1.3k, Resistor_SMD:R_0805_2012Metric
- removed R19: 23.7k, Resistor_SMD:R_0805_2012Metric
- removed R20: 374k, Resistor_SMD:R_0805_2012Metric
- removed R22: 100k, Resistor_SMD:R_0805_2012Metric
- removed R23: 1.07M, Resistor_SMD:R_0805_2012Metric
- removed R24: 120k, Resistor_SMD:R_0805_2012Metric
- removed R25, R26, R31, R32: 10k, Resistor_SMD:R_0805_2012Metric
- removed R27, R28, R29, R30, R33, R34: 1k, Resistor_SMD:R_0805_2012Metric
- removed R38, R39, R40, R41, R42, R43, R44: 5k, Resistor_SMD:R_0805_2012Metric
- removed U10, U11, U8: ADS1115IDGS, Package_SO:TSSOP-10_3x3mm_P0.5mm
- removed U21: TPS61089, Package_DFN_QFN:Texas_VQFN-RNR0011A-11
- removed U22: TPS7A4701xRGW, Package_DFN_QFN:Texas_RGW0020A_VQFN-20-1EP_5x5mm_P0.65mm_EP3.15x3.15mm
- moved J34 356.5 mm to (466.0, 104.4), turned to -120 degrees
- moved J35 351.7 mm to (448.2, 57.7), turned to -60 degrees
- moved J25 330.6 mm to (458.5, 117.8), turned to -120 degrees
- moved J5 329.4 mm to (455.9, 71.0), turned to -60 degrees
- moved J12 321.4 mm to (434.8, 143.0), turned to 180 degrees
- moved J15 313.1 mm to (470.0, 97.1), turned to -120 degrees
- moved J7 294.1 mm to (399.0, 49.8)
- moved J4 290.6 mm to (414.2, 49.8)
- moved J10 289.5 mm to (444.1, 50.4), turned to -60 degrees
- moved J24 289.3 mm to (419.4, 143.0), turned to 180 degrees
- moved J2 283.5 mm to (390.2, 50.0), turned to 60 degrees
- moved J13 282.3 mm to (442.9, 143.0), turned to 180 degrees
- moved J33 275.6 mm to (378.1, 70.5), turned to 60 degrees
- moved J9 262.0 mm to (375.1, 116.8), turned to 120 degrees
- moved J23 259.5 mm to (389.6, 142.4), turned to 120 degrees
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Connections:
- J3 pad 5: TEMP_SCL -> TEMP_SDA
- U1 pad 94: TEMP_SCL -> TEMP_SDA
- U9 pad 21: GPIO_A0 -> GPIO_A7
- U9 pad 22: GPIO_A1 -> GPIO_A6
- U9 pad 23: GPIO_A2 -> GPIO_A5
- U9 pad 24: GPIO_A3 -> GPIO_A4
- U9 pad 25: GPIO_A4 -> GPIO_A3
- U9 pad 26: GPIO_A5 -> GPIO_A2
- U9 pad 27: GPIO_A6 -> GPIO_A1
- U9 pad 28: GPIO_A7 -> GPIO_A0
Other:
- board text added: ":)"
