File: Aurora_new/_autosave-Aurora.kicad_pcb (KiCad board)
At the start: 2 copper layers, 129 parts, among them J1 UJ20-C-H-C-3-SMT-TR, J10 Screw_Terminal_01x02, J11 Screw_Terminal_01x02, J12 Screw_Terminal_01x04, J13 Screw_Terminal_01x02, J14 Screw_Terminal_01x02, J15 Screw_Terminal_01x02, J16 PPPC042LFBN-RC, J2 Screw_Terminal_01x04, J22 Screw_Terminal_01x08, J23 Screw_Terminal_01x08, J24 Screw_Terminal_01x08, J25 Screw_Terminal_01x08, J3 PPPC042LFBN-RC, J33 Screw_Terminal_01x04, J34 Screw_Terminal_01x04, J35 Screw_Terminal_01x04, J36 PPPC042LFBN-RC, J4 Screw_Terminal_01x08, J41 STEMMA QT, J49 PPTC032LFBN-RC, J5 Screw_Terminal_01x08, J50 PCB.RPSMAFRA.HT, J52 PPTC041LFBN-RC, J6 DM3AT-SF-PEJM5, J7 Screw_Terminal_01x04, J9 Screw_Terminal_01x04, Q9 FMMT619TA, U1 STM32H757BITx, U12 XBP9X-DMRS-001, U14 MS5611-01BA, U15 TPS7A4701xRGW, U17 MCP1826ST-3302E/DB, U18 MCP1826ST-3302E/DB, U19 MCP1826ST-3302E/DB, U2 USBLC6-2SC6, U20 TPS7A4701xRGW, U3 TPS2121RUXR, U4 TPS7A4701xRGW, U5 ICM-45686, U6 ICM-42688-P, U7 BNO085, U9 MCP23017T-E_SO

Commit message: layout and changed screw term size
Parts:
- removed J2: Screw_Terminal_01x04, 1984633:PHOENIX_1984633
- added J17: Screw_Terminal_01x02, 1725656:PHOENIX_1725656, F.Cu at (407.5, 79.1)
- added J8: Screw_Terminal_01x02, 1725656:PHOENIX_1725656, F.Cu at (397.8, 27.6)
- J10, J11, J13, J14, J15: footprint 1984617:PHOENIX_1984617 -> 1725656:PHOENIX_1725656
- J12, J33, J34, J35, J7, J9: footprint 1984633:PHOENIX_1984633 -> 1725672:PHOENIX_1725672
- J22, J23, J24, J25, J4, J5: footprint 1984675:PHOENIX_1984675 -> 1725711:PHOENIX_1725711
- moved J1 385.9 mm to (473.2, 87.8), turned to 90 degrees
- moved J5 293.5 mm to (455.7, 55.3), turned to -60 degrees
- moved J25 284.5 mm to (458.5, 117.8), turned to -120 degrees
- moved J4 253.6 mm to (430.3, 27.6), turned to 180 degrees
- moved J34 246.3 mm to (466.0, 104.4), turned to -120 degrees
- moved J24 245.2 mm to (419.4, 143.0), turned to 180 degrees
- moved J35 241.9 mm to (448.0, 42.0), turned to -60 degrees
- moved J15 239.7 mm to (470.0, 97.1), turned to -120 degrees
- moved J7 220.2 mm to (408.9, 27.6), turned to 180 degrees
- moved J10 208.1 mm to (443.9, 34.6), turned to -60 degrees
- moved J12 201.8 mm to (434.8, 143.0), turned to 180 degrees
- moved J22 199.4 mm to (363.3, 80.2), turned to 60 degrees
- moved J13 188.9 mm to (442.9, 143.0), turned to 180 degrees
- moved J11 141.1 mm to (385.6, 41.5), turned to 60 degrees
- moved J14 130.6 mm to (367.4, 103.6), turned to 120 degrees
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Connections:
- U9 pad 21: GPIO_A0 -> GPIO_A7
- U9 pad 22: GPIO_A1 -> GPIO_A6
- U9 pad 23: GPIO_A2 -> GPIO_A5
- U9 pad 24: GPIO_A3 -> GPIO_A4
- U9 pad 25: GPIO_A4 -> GPIO_A3
- U9 pad 26: GPIO_A5 -> GPIO_A2
- U9 pad 27: GPIO_A6 -> GPIO_A1
- U9 pad 28: GPIO_A7 -> GPIO_A0
Other:
- board text added: ":)"
